Commit message: update11.5

File: description/gazebo_control.xacro (robot description, xacro)
@@ -2,20 +2,21 @@
 <robot xmlns:xacro="http://www.ros.org/wiki/xacro">
     <gazebo>
-        <plugin name="gz::sim::systems::DiffDrive" filename="gz-sim-diff-drive-system">
-            <!-- Wheel Information -->
+        <plugin name="gz::sim::systems::DiffDrive"
+                filename="gz-sim-diff-drive-system">
             <left_joint>left_wheel_joint</left_joint>
             <right_joint>right_wheel_joint</right_joint>
             <wheel_separation>0.35</wheel_separation>
             <wheel_radius>0.1</wheel_radius>
-            <!-- Input -->
-            <topic>cmd_vel</topic>
-            <!-- Output -->
+            <topic>/cmd_vel</topic>
             <frame_id>odom</frame_id>
             <child_frame_id>base_link</child_frame_id>
-            <odom_topic>odom</odom_topic>
-            <tf_topic>tf</tf_topic>
+            <odom_topic>/odom</odom_topic>
+            <tf_topic>/tf</tf_topic>
+            <odom_publish_frequency>30</odom_publish_frequency>
+            <max_linear_acceleration>10</max_linear_acceleration>
         </plugin>
-        <plugin name="gz::sim::systems::JointStatePublisher" filename="gz-sim-joint-state-publisher-system">
-            <topic>joint_states</topic>
+        <plugin name="gz::sim::systems::JointStatePublisher"
+                filename="gz-sim-joint-state-publisher-system">
+            <topic>/joint_state</topic>
             <joint_name>left_wheel_joint</joint_name>
             <joint_name>right_wheel_joint</joint_name>

File: description/robot_core.xacro (robot description, xacro)
@@ -13,4 +13,7 @@
     <material name="black">
         <color rgba="0 0 0 1"/>
+    </material>
+    <material name="red">
+        <color rgba="1 0 0 1"/>
     </material>
     <!--BASE LINK-->
@@ -41,6 +44,11 @@
         </xacro:inertial_box>
     </link>
-    <gazebo reference ="chassis">
-        <material>Gazebo/white</material>
+    <gazebo reference="chassis">
+        <visual>
+            <material>
+                <ambient>1 1 1 1</ambient>
+                <diffuse>1 1 1 1</diffuse>
+            </material>
+        </visual>
     </gazebo>
     <!-- LEFT WHEEL -->
@@ -50,4 +58,5 @@
         <origin xyz="0 0.175 0" rpy="-${pi/2} 0 0"/>
         <axis xyz="0 0 1"/>
+        <limit effort="10.0" velocity="10.0"/>
     </joint>
     <link name="left_wheel">
@@ -68,5 +77,10 @@
     </link>
     <gazebo reference ="left_wheel">
-        <material>Gazebo/Blue</material>
+        <visual>
+            <material>
+                <ambient>0.2 0.2 1 1</ambient>
+                <diffuse>0.2 0.2 1 1</diffuse>
+            </material>
+        </visual>
     </gazebo>
     <!-- RIGHT WHEEL -->
@@ -76,4 +90,5 @@
         <origin xyz="0 -0.175 0" rpy="${pi/2} 0 0"/>
         <axis xyz="0 0 -1"/>
+        <limit effort="10.0" velocity="10.0"/>
     </joint>
     <link name="right_wheel">
@@ -94,5 +109,10 @@
     </link>
     <gazebo reference ="right_wheel">
-        <material>Gazebo/Blue</material>
+        <visual>
+            <material>
+                <ambient>0.2 0.2 1 1</ambient>
+                <diffuse>0.2 0.2 1 1</diffuse>
+            </material>
+        </visual>
     </gazebo>
     <!-- CASTER WHEEL -->
@@ -118,6 +138,11 @@
         </xacro:inertial_sphere>
     </link>
-    <gazebo reference ="caster_wheel">
-        <material>Gazebo/Black</material>
+    <gazebo reference="caster_wheel">
+        <visual>
+            <material>
+                <ambient>0 0 0 1</ambient>
+                <diffuse>0 0 0 1</diffuse>
+            </material>
+        </visual>
         <mu1 value="0.001"/>
         <mu2 value="0.001"/>
